File: power.brd (EAGLE design)
At the start: 83 x 56 mm, 10 parts

Commit message: slightly modified logo position
Parts:
- moved LOGO1 2.65 mm to (62.6, 5.50)
Changed lines of the file:
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@@
 <element name="STANDOFF7" library="SparkFun-Electromechanical" package="STAND-OFF" value="STAND-OFF" x="11" y="13"/>
 <element name="STANDOFF8" library="SparkFun-Electromechanical" package="STAND-OFF" value="STAND-OFF" x="41" y="43"/>
-<element name="LOGO1" library="SparkFun-Aesthetics" package="OSHW-LOGO-L" value="OSHW-LOGOL" x="60" y="6"/>
+<element name="LOGO1" library="SparkFun-Aesthetics" package="OSHW-LOGO-L" value="OSHW-LOGOL" x="62.6" y="5.5"/>
 </elements>
 <signals>

Commit message: build up the frame work
Parts:
- added JP1, JP2, JP3, JP4, JP5, JP6, JP7, JP8: M01SMD-6X3, SparkFun-Connectors-modified:PAD-BULLET
- moved FRAME1 13.0 mm to (22.0, -21.0)
Other:
- outline, holes or cut-outs redrawn
Changed lines of the file:
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@@
 <layer number="111" name="LPC17xx" color="7" fill="1" visible="yes" active="yes"/>
 <layer number="112" name="tSilk" color="7" fill="1" visible="yes" active="yes"/>
+<layer number="113" name="IDFDebug" color="4" fill="1" visible="no" active="yes"/>
 <layer number="116" name="Patch_BOT" color="9" fill="4" visible="yes" active="yes"/>
 <layer number="121" name="_tsilk" color="7" fill="1" visible="yes" active="yes"/>
@@
 <wire x1="68" y1="56" x2="83" y2="53" width="0" layer="20"/>
 <wire x1="68" y1="0" x2="83" y2="3" width="0" layer="20"/>
-<wire x1="11" y1="17" x2="41" y2="17" width="0" layer="20"/>
-<wire x1="11" y1="17" x2="11" y2="39" width="0" layer="20"/>
-<wire x1="41" y1="39" x2="11" y2="39" width="0" layer="20"/>
-<wire x1="41" y1="39" x2="41" y2="17" width="0" layer="20"/>
+<wire x1="11" y1="23" x2="41" y2="23" width="0" layer="20"/>
+<wire x1="11" y1="23" x2="11" y2="33" width="0" layer="20"/>
+<wire x1="41" y1="33" x2="11" y2="33" width="0" layer="20"/>
+<wire x1="41" y1="33" x2="41" y2="23" width="0" layer="20"/>
 <wire x1="48.5" y1="43" x2="48.5" y2="13" width="0" layer="20"/>
 <wire x1="48.5" y1="43" x2="57" y2="43" width="0" layer="20"/>
@@
 <wire x1="76" y1="49" x2="76" y2="7" width="0" layer="20"/>
 <wire x1="68" y1="7" x2="76" y2="7" width="0" layer="20"/>
-<text x="48" y="-8" size="1.778" layer="51">Librae</text>
+<text x="49" y="-21" size="1.778" layer="51">Librae</text>
+<wire x1="10" y1="6" x2="10" y2="-11" width="0.254" layer="51"/>
+<wire x1="15" y1="6" x2="15" y2="-11" width="0.254" layer="51"/>
+<wire x1="10" y1="6" x2="15" y2="6" width="0.254" layer="51"/>
+<wire x1="10" y1="-11" x2="15" y2="-11" width="0.254" layer="51"/>
+<wire x1="20" y1="6" x2="20" y2="-11" width="0.254" layer="51"/>
+<wire x1="25" y1="6" x2="25" y2="-11" width="0.254" layer="51"/>
+<wire x1="20" y1="6" x2="25" y2="6" width="0.254" layer="51"/>
+<wire x1="20" y1="-11" x2="25" y2="-11" width="0.254" layer="51"/>
+<wire x1="27" y1="6" x2="27" y2="-11" width="0.254" layer="51"/>
+<wire x1="32" y1="6" x2="32" y2="-11" width="0.254" layer="51"/>
+<wire x1="27" y1="6" x2="32" y2="6" width="0.254" layer="51"/>
+<wire x1="27" y1="-11" x2="32" y2="-11" width="0.254" layer="51"/>
+<wire x1="37" y1="6" x2="37" y2="-11" width="0.254" layer="51"/>
+<wire x1="42" y1="6" x2="42" y2="-11" width="0.254" layer="51"/>
+<wire x1="37" y1="6" x2="42" y2="6" width="0.254" layer="51"/>
+<wire x1="37" y1="-11" x2="42" y2="-11" width="0.254" layer="51"/>
+<wire x1="10" y1="67" x2="10" y2="50" width="0.254" layer="51"/>
+<wire x1="15" y1="67" x2="15" y2="50" width="0.254" layer="51"/>
+<wire x1="10" y1="67" x2="15" y2="67" width="0.254" layer="51"/>
+<wire x1="10" y1="50" x2="15" y2="50" width="0.254" layer="51"/>
+<wire x1="20" y1="67" x2="20" y2="50" width="0.254" layer="51"/>
+<wire x1="25" y1="67" x2="25" y2="50" width="0.254" layer="51"/>
+<wire x1="20" y1="67" x2="25" y2="67" width="0.254" layer="51"/>
+<wire x1="20" y1="50" x2="25" y2="50" width="0.254" layer="51"/>
+<wire x1="27" y1="67" x2="27" y2="50" width="0.254" layer="51"/>
+<wire x1="32" y1="67" x2="32" y2="50" width="0.254" layer="51"/>
+<wire x1="27" y1="67" x2="32" y2="67" width="0.254" layer="51"/>
+<wire x1="27" y1="50" x2="32" y2="50" width="0.254" layer="51"/>
+<wire x1="37" y1="67" x2="37" y2="50" width="0.254" layer="51"/>
+<wire x1="42" y1="67" x2="42" y2="50" width="0.254" layer="51"/>
+<wire x1="37" y1="67" x2="42" y2="67" width="0.254" layer="51"/>
+<wire x1="37" y1="50" x2="42" y2="50" width="0.254" layer="51"/>
+<wire x1="0.5" y1="10" x2="50.5" y2="10" width="0.254" layer="51"/>
+<wire x1="0.5" y1="10" x2="0.5" y2="46" width="0.254" layer="51"/>
+<wire x1="0.5" y1="46" x2="50.5" y2="46" width="0.254" layer="51"/>
+<wire x1="50.5" y1="10" x2="50.5" y2="46" width="0.254" layer="51"/>
 </plain>
 <attributes>
@@
 </autorouter>
 <elements>
-<element name="FRAME1" library="SparkFun-Aesthetics" package="CREATIVE_COMMONS" value="FRAME-LETTER" x="21" y="-8"/>
+<element name="FRAME1" library="SparkFun-Aesthetics" package="CREATIVE_COMMONS" value="FRAME-LETTER" x="22" y="-21"/>
 <element name="STANDOFF1" library="SparkFun-Electromechanical" package="STAND-OFF" value="STAND-OFF" x="3.5" y="50.5"/>
 <element name="STANDOFF2" library="SparkFun-Electromechanical" package="STAND-OFF" value="STAND-OFF" x="48.5" y="5.5"/>
@@
 <element name="STANDOFF8" library="SparkFun-Electromechanical" package="STAND-OFF" value="STAND-OFF" x="41" y="43"/>
 <element name="LOGO1" library="SparkFun-Aesthetics" package="OSHW-LOGO-L" value="OSHW-LOGOL" x="62.6" y="5.5"/>
+<element name="JP1" library="SparkFun-Connectors-modified" package="PAD-BULLET" value="M01SMD-6X3" x="12.5" y="52.5" rot="R270"/>
+<element name="JP2" library="SparkFun-Connectors-modified" package="PAD-BULLET" value="M01SMD-6X3" x="22.5" y="52.5" rot="R90"/>
+<element name="JP3" library="SparkFun-Connectors-modified" package="PAD-BULLET" value="M01SMD-6X3" x="39.5" y="3.5" rot="R90"/>
+<element name="JP4" library="SparkFun-Connectors-modified" package="PAD-BULLET" value="M01SMD-6X3" x="29.5" y="3.5" rot="R90"/>
+<element name="JP5" library="SparkFun-Connectors-modified" package="PAD-BULLET" value="M01SMD-6X3" x="12.5" y="3.5" rot="R90"/>
+<element name="JP6" library="SparkFun-Connectors-modified" package="PAD-BULLET" value="M01SMD-6X3" x="22.5" y="3.5" rot="R90"/>
+<element name="JP7" library="SparkFun-Connectors-modified" package="PAD-BULLET" value="M01SMD-6X3" x="39.5" y="52.5" rot="R90"/>
+<element name="JP8" library="SparkFun-Connectors-modified" package="PAD-BULLET" value="M01SMD-6X3" x="29.5" y="52.5" rot="R90"/>
 </elements>
 <signals>

Commit message: update layout
Parts:
- added JP10, JP11, JP12, JP9: M01SMD-6X3, SparkFun-Connectors-modified:PAD-BULLET
- moved LOGO1 1.00 mm to (61.6, 5.50)
Connections:
- new net GND: JP10.P$1, JP12.P$1, JP2.P$1, JP4.P$1, JP6.P$1, JP8.P$1
- new net VIN: JP1.P$1, JP11.P$1, JP3.P$1, JP5.P$1, JP7.P$1, JP9.P$1
Routing:
- net VIN: track 0.00 -> 363.5 mm
- net GND: track 0.00 -> 93.5 mm, vias 0 -> 136
- added copper zone on layer 1, net GND
- added copper zone on layer 16, net GND
Other:
- outline, holes or cut-outs redrawn
