File: power.brd (EAGLE design)
At the start: 83 x 56 mm, 22 parts

Commit message: almost done
Parts:
- added JP13: (no value), SparkFun-Connectors:1X03_LONGPADS
- added JP14: M02PTH3, SparkFun-Connectors:1X02_LONGPADS
- added S2: SWITCH-MOMENTARY-2PTH-2, SparkFun-Electromechanical:TACTILE-PTH-2
- added SAFETY: (no value), adafruit:1206
- added SG1: BUZZERNS, SparkFun-Electromechanical:BUZZER-12MM-NS
- moved LOGO1 20.3 mm to (76.5, 46.5)
Connections:
- new net 3.3V: JP13.1, S2.4, SAFETY.A
- new net N$3: JP14.1, SG1.+
- new net N$4: JP13.3, S2.1
- new net N$5: JP13.2, SAFETY.C
- new net N$6: JP14.2, SG1.-
Routing:
- net 3.3V: track 0.00 -> 43.7 mm
- net N$3: track 0.00 -> 29.9 mm
- net N$5: track 0.00 -> 21.4 mm
- net N$6: track 0.00 -> 19.4 mm
- net N$4: track 0.00 -> 7.86 mm
- net VIN: track 401.7 -> 409.2 mm
Other:
- outline, holes or cut-outs redrawn
Changed lines of the file:
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@@
 <setting verticaltext="up"/>
 </settings>
-<grid distance="0.5" unitdist="mm" unit="mm" style="lines" multiple="1" display="yes" altdistance="0.05" altunitdist="mm" altunit="mm"/>
+<grid distance="0.0196850394" unitdist="inch" unit="inch" style="lines" multiple="1" display="yes" altdistance="0.05" altunitdist="mm" altunit="mm"/>
 <layers>
 <layer number="1" name="Top" color="4" fill="1" visible="yes" active="yes"/>
@@
 <wire x1="68" y1="56" x2="0" y2="56" width="0" layer="20"/>
 <wire x1="0" y1="56" x2="0" y2="0" width="0" layer="20"/>
-<wire x1="83" y1="53" x2="83" y2="3" width="0" layer="20"/>
-<wire x1="68" y1="56" x2="83" y2="53" width="0" layer="20"/>
+<wire x1="68" y1="56" x2="76" y2="54.4" width="0" layer="20"/>
+<wire x1="76" y1="54.4" x2="83" y2="53" width="0" layer="20" style="longdash"/>
 <wire x1="68" y1="0" x2="83" y2="3" width="0" layer="20"/>
 <wire x1="55.5" y1="43" x2="55.5" y2="13" width="0" layer="20"/>
@@
 <wire x1="61.5" y1="43" x2="61.5" y2="13" width="0" layer="20"/>
 <wire x1="55.5" y1="13" x2="61.5" y2="13" width="0" layer="20"/>
-<wire x1="68" y1="49" x2="68" y2="7" width="0" layer="20"/>
-<wire x1="68" y1="49" x2="76" y2="49" width="0" layer="20"/>
-<wire x1="76" y1="49" x2="76" y2="7" width="0" layer="20"/>
-<wire x1="68" y1="7" x2="76" y2="7" width="0" layer="20"/>
+<wire x1="83" y1="40" x2="70" y2="40" width="0" layer="20"/>
+<wire x1="70" y1="40" x2="70" y2="16" width="0" layer="20"/>
+<wire x1="70" y1="16" x2="83" y2="16" width="0" layer="20"/>
 <text x="49" y="-21" size="1.778" layer="51">Librae</text>
 <wire x1="10" y1="4" x2="10" y2="-10" width="0.254" layer="51"/>
@@
 <wire x1="4.5" y1="41" x2="4.5" y2="39" width="0.4064" layer="21"/>
 <wire x1="4.5" y1="15" x2="4.5" y2="17" width="0.4064" layer="22"/>
-<wire x1="0" y1="28" x2="26" y2="28" width="0.254" layer="37"/>
-<wire x1="26" y1="28" x2="34" y2="28" width="0.254" layer="37"/>
+<wire x1="25.5" y1="28" x2="26" y2="28" width="0.254" layer="37"/>
+<wire x1="26" y1="28" x2="26.5" y2="28" width="0.254" layer="37"/>
+<wire x1="33.5" y1="28" x2="34" y2="28" width="0.254" layer="37"/>
 <wire x1="34" y1="28" x2="34" y2="27.5" width="0.254" layer="37"/>
 <wire x1="34" y1="28" x2="34" y2="28.5" width="0.254" layer="37"/>
-<wire x1="34" y1="28" x2="83" y2="28" width="0.254" layer="37"/>
+<wire x1="34" y1="28" x2="34.5" y2="28" width="0.254" layer="37"/>
 <wire x1="26" y1="28" x2="26" y2="28.5" width="0.254" layer="37"/>
 <wire x1="26" y1="28" x2="26" y2="27.5" width="0.254" layer="37"/>
@@
 <wire x1="58.5" y1="45.5" x2="68.5" y2="45.5" width="0.254" layer="51"/>
 <wire x1="58.5" y1="10.5" x2="68.5" y2="10.5" width="0.254" layer="51"/>
+<wire x1="83" y1="53" x2="83" y2="40" width="0" layer="20"/>
+<wire x1="83" y1="3" x2="83" y2="16" width="0" layer="20"/>
+<wire x1="54.5" y1="4.5" x2="54.5" y2="2.5" width="0.4064" layer="21"/>
+<wire x1="53.5" y1="3.5" x2="55.5" y2="3.5" width="0.4064" layer="21"/>
+<wire x1="58" y1="3.5" x2="60" y2="3.5" width="0.4064" layer="21"/>
 </plain>
 <attributes>
@@
 <element name="STANDOFF7" library="SparkFun-Electromechanical" package="STAND-OFF" value="STAND-OFF" x="19" y="13"/>
 <element name="STANDOFF8" library="SparkFun-Electromechanical" package="STAND-OFF" value="STAND-OFF" x="49" y="43"/>
-<element name="LOGO1" library="SparkFun-Aesthetics" package="OSHW-LOGO-L" value="OSHW-LOGOL" x="56.6" y="50.5"/>
+<element name="LOGO1" library="SparkFun-Aesthetics" package="OSHW-LOGO-L" value="OSHW-LOGOL" x="76.5" y="46.5"/>
 <element name="JP1" library="SparkFun-Connectors-modified" package="PAD-BULLET" value="M01SMD-6X3" x="12.5" y="52.5" rot="R270"/>
 <element name="JP2" library="SparkFun-Connectors-modified" package="PAD-BULLET" value="M01SMD-6X3" x="22.5" y="52.5" rot="R90"/>
@@
 <element name="JP11" library="SparkFun-Connectors-modified" package="PAD-BULLET" value="M01SMD-6X3" x="7.5" y="34" rot="R270"/>
 <element name="JP12" library="SparkFun-Connectors-modified" package="PAD-BULLET" value="M01SMD-6X3" x="7.5" y="22" rot="MR90"/>
+<element name="SG1" library="SparkFun-Electromechanical" package="BUZZER-12MM-NS" value="BUZZERNS" x="75.5" y="9"/>
+<element name="SAFETY" library="adafruit" package="1206" value="" x="76.5" y="46.5" rot="R180"/>
+<element name="S2" library="SparkFun-Electromechanical" package="TACTILE-PTH-2" value="SWITCH-MOMENTARY-2PTH-2" x="65.5" y="50.5" rot="R270"/>
+<element name="JP13" library="SparkFun-Connectors" package="1X03_LONGPADS" value="" x="54.5" y="49"/>
+<element name="JP14" library="SparkFun-Connectors" package="1X02_LONGPADS" value="M02PTH3" x="55.5" y="7"/>
 </elements>
 <signals>
@@
 <wire x1="8" y1="22" x2="8" y2="33.5" width="3.81" layer="1"/>
 <wire x1="8" y1="33.5" x2="7.5" y2="34" width="3.81" layer="1"/>
-<wire x1="12.5" y1="52.5" x2="12.5" y2="51" width="3.81" layer="1"/>
-<wire x1="12.5" y1="51" x2="4.5" y2="43" width="3.81" layer="1"/>
-<wire x1="4.5" y1="43" x2="4.5" y2="34" width="3.81" layer="1"/>
+<wire x1="12.5" y1="52.5" x2="12.5" y2="50.5" width="3.81" layer="1"/>
+<wire x1="12.5" y1="50.5" x2="4.5" y2="42.5" width="3.81" layer="1"/>
+<wire x1="4.5" y1="42.5" x2="4.5" y2="34" width="3.81" layer="1"/>
 <wire x1="4.5" y1="34" x2="3.75" y2="33.25" width="3.81" layer="1"/>
 <wire x1="3.75" y1="33.25" x2="3.25" y2="33.25" width="3.81" layer="1"/>
@@
 <wire x1="4.5" y1="13.5" x2="12.5" y2="5.5" width="3.81" layer="1"/>
 <wire x1="12.5" y1="3" x2="12.5" y2="3.5" width="3.81" layer="1"/>
-<wire x1="12.5" y1="3.5" x2="12.5" y2="5.5" width="3.81" layer="1"/>
+<wire x1="12.5" y1="3.5" x2="12.5" y2="4" width="3.81" layer="1"/>
+<wire x1="12.5" y1="4" x2="12.5" y2="5.5" width="3.81" layer="1"/>
 <wire x1="39.5" y1="11.5" x2="39.5" y2="16" width="3.81" layer="1"/>
 <wire x1="39.5" y1="52.5" x2="38" y2="41.5" width="3.81" layer="1"/>
@@
 <wire x1="8" y1="22" x2="12.5" y2="26.5" width="3.81" layer="1"/>
 <wire x1="7.5" y1="35.5" x2="7.5" y2="34.5" width="3.81" layer="1"/>
-<wire x1="7.5" y1="34.5" x2="11" y2="31" width="3.81" layer="1"/>
-<wire x1="12.5" y1="53.5" x2="11" y2="53.5" width="0" layer="19" extent="1-1"/>
-<wire x1="7.5" y1="34.5" x2="7.5" y2="34" width="0" layer="19" extent="1-1"/>
-<wire x1="46.5" y1="29" x2="46.5" y2="28.5" width="0" layer="19" extent="1-1"/>
-<wire x1="11" y1="2.5" x2="12.5" y2="3" width="0" layer="19" extent="1-1"/>
+<wire x1="7.5" y1="34.5" x2="8" y2="34" width="3.81" layer="1"/>
+<wire x1="8" y1="34" x2="11" y2="31" width="3.81" layer="1"/>
+<wire x1="46.5" y1="28.5" x2="46.5" y2="29" width="0.254" layer="1"/>
+<wire x1="7.5" y1="34" x2="8" y2="34" width="0.254" layer="1"/>
+<wire x1="11" y1="2.5" x2="12.5" y2="2.5" width="0.254" layer="1"/>
+<wire x1="12.5" y1="2.5" x2="12.5" y2="4" width="0.254" layer="1"/>
+<wire x1="12.5" y1="53.5" x2="13" y2="53.5" width="0.254" layer="1"/>
+<wire x1="13" y1="53.5" x2="13" y2="52" width="0.254" layer="1"/>
+<wire x1="12.5" y1="53.5" x2="11" y2="53.5" width="0.254" layer="1"/>
 </signal>
 <signal name="GND">
@@
 <wire x1="41" y1="53.5" x2="41" y2="43.5" width="3.81" layer="1"/>
 </signal>
+<signal name="3.3V">
+<contactref element="SAFETY" pad="A"/>
+<contactref element="JP13" pad="1"/>
+<contactref element="S2" pad="4"/>
+<wire x1="54.5" y1="49" x2="54.5" y2="45.5" width="0.4064" layer="1"/>
+<wire x1="54.5" y1="45.5" x2="55.5" y2="44.5" width="0.4064" layer="1"/>
+<wire x1="55.5" y1="44.5" x2="77" y2="44.5" width="0.4064" layer="1"/>
+<wire x1="77" y1="44.5" x2="78" y2="45.5" width="0.4064" layer="1"/>
+<wire x1="78" y1="45.5" x2="78" y2="46.422" width="0.4064" layer="1"/>
+<wire x1="78" y1="46.422" x2="77.922" y2="46.5" width="0.4064" layer="1"/>
+<wire x1="65.5" y1="47.325" x2="68.825" y2="47.325" width="0.4064" layer="1"/>
+<wire x1="68.825" y1="47.325" x2="70.5" y2="49" width="0.4064" layer="1"/>
+<wire x1="70.5" y1="49" x2="76.5" y2="49" width="0.4064" layer="1"/>
+<wire x1="76.5" y1="49" x2="78" y2="47.5" width="0.4064" layer="1"/>
+<wire x1="78" y1="47.5" x2="78" y2="46.578" width="0.4064" layer="1"/>
+<wire x1="78" y1="46.578" x2="77.922" y2="46.5" width="0.4064" layer="1"/>
+</signal>
+<signal name="N$5">
+<contactref element="SAFETY" pad="C"/>
+<contactref element="JP13" pad="2"/>
+<wire x1="57.04" y1="49" x2="57.04" y2="46.46" width="0.4064" layer="1"/>
+<wire x1="57.04" y1="46.46" x2="58" y2="45.5" width="0.4064" layer="1"/>
+<wire x1="58" y1="45.5" x2="71" y2="45.5" width="0.4064" layer="1"/>
+<wire x1="71" y1="45.5" x2="72" y2="46.5" width="0.4064" layer="1"/>
+<wire x1="72" y1="46.5" x2="75.078" y2="46.5" width="0.4064" layer="1"/>
+</signal>
+<signal name="N$6">
+<contactref element="SG1" pad="-"/>
+<contactref element="JP14" pad="2"/>
+<wire x1="58.04" y1="7" x2="58.04" y2="4.46" width="0.4064" layer="1"/>
+<wire x1="58.04" y1="4.46" x2="59" y2="3.5" width="0.4064" layer="1"/>
+<wire x1="59" y1="3.5" x2="66.75" y2="3.5" width="0.4064" layer="1"/>
+<wire x1="66.75" y1="3.5" x2="72.25" y2="9" width="0.4064" layer="1"/>
+</signal>
+<signal name="N$3">
+<contactref element="JP14" pad="1"/>
+<contactref element="SG1" pad="+"/>
+<wire x1="55.5" y1="7" x2="55.5" y2="3.5" width="0.4064" layer="1"/>
+<wire x1="55.5" y1="3.5" x2="56.5" y2="2.5" width="0.4064" layer="1"/>
+<wire x1="56.5" y1="2.5" x2="72.25" y2="2.5" width="0.4064" layer="1"/>
+<wire x1="72.25" y1="2.5" x2="78.75" y2="9" width="0.4064" layer="1"/>
+</signal>
+<signal name="N$4">
+<contactref element="JP13" pad="3"/>
+<contactref element="S2" pad="1"/>
+<wire x1="59.58" y1="49" x2="64.255" y2="53.675" width="0.4064" layer="1"/>
+<wire x1="64.255" y1="53.675" x2="65.5" y2="53.675" width="0.4064" layer="1"/>
+</signal>
 </signals>

Commit message: basically done
Parts:
- added JP15, JP16: M01SMD, SparkFun-Connectors-modified:LUXEON-PAD
- SAFETY: device adafruit:1206 -> adafruit:LED5MM
- moved LOGO1 43.1 mm to (65.0, 5.00)
- moved SG1 0.50 mm to (76.0, 9.00), turned to 270 degrees
Connections:
- net N$3: now also JP16.P$1
- net N$5: now also SAFETY.K; no longer SAFETY.C
- net N$6: now also JP15.P$1
Routing:
- net VIN: track 409.2 -> 396.1 mm
- net N$6: track 19.4 -> 29.5 mm
- net N$3: track 29.9 -> 30.8 mm
- net GND: vias 84 -> 86
