File: power.sch (EAGLE design)
At the start: 10 parts

Commit message: build up the frame work
Parts:
- added JP1, JP2, JP3, JP4, JP5, JP6, JP7, JP8: M01SMD-6X3, SparkFun-Connectors-modified:M01SMD-6X3
Changed lines of the file:
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@@
 <setting verticaltext="up"/>
 </settings>
-<grid distance="0.1" unitdist="inch" unit="inch" style="lines" multiple="1" display="no" altdistance="0.01" altunitdist="inch" altunit="inch"/>
+<grid distance="0.1" unitdist="inch" unit="inch" style="lines" multiple="1" display="yes" altdistance="0.01" altunitdist="inch" altunit="inch"/>
 <layers>
 <layer number="1" name="Top" color="4" fill="1" visible="no" active="no"/>
@@
 <layer number="111" name="LPC17xx" color="7" fill="1" visible="yes" active="yes"/>
 <layer number="112" name="tSilk" color="7" fill="1" visible="yes" active="yes"/>
+<layer number="113" name="IDFDebug" color="4" fill="1" visible="no" active="yes"/>
 <layer number="116" name="Patch_BOT" color="9" fill="4" visible="yes" active="yes"/>
 <layer number="121" name="_tsilk" color="7" fill="1" visible="yes" active="yes"/>
@@
 <part name="STANDOFF8" library="SparkFun-Electromechanical" deviceset="STAND-OFF" device=""/>
 <part name="LOGO1" library="SparkFun-Aesthetics" deviceset="OSHW-LOGO" device="L"/>
+<part name="JP1" library="SparkFun-Connectors-modified" deviceset="M01" device="SMD-6X3"/>
+<part name="JP2" library="SparkFun-Connectors-modified" deviceset="M01" device="SMD-6X3"/>
+<part name="JP3" library="SparkFun-Connectors-modified" deviceset="M01" device="SMD-6X3"/>
+<part name="JP4" library="SparkFun-Connectors-modified" deviceset="M01" device="SMD-6X3"/>
+<part name="JP5" library="SparkFun-Connectors-modified" deviceset="M01" device="SMD-6X3"/>
+<part name="JP6" library="SparkFun-Connectors-modified" deviceset="M01" device="SMD-6X3"/>
+<part name="JP7" library="SparkFun-Connectors-modified" deviceset="M01" device="SMD-6X3"/>
+<part name="JP8" library="SparkFun-Connectors-modified" deviceset="M01" device="SMD-6X3"/>
 </parts>
 <sheets>
@@
 <instance part="STANDOFF8" gate="G$1" x="71.12" y="104.14"/>
 <instance part="LOGO1" gate="G$1" x="129.54" y="20.32"/>
+<instance part="JP1" gate="G$1" x="101.6" y="124.46" rot="R90"/>
+<instance part="JP2" gate="G$1" x="111.76" y="124.46" rot="R90"/>
+<instance part="JP3" gate="G$1" x="165.1" y="88.9" rot="R270"/>
+<instance part="JP4" gate="G$1" x="154.94" y="88.9" rot="R270"/>
+<instance part="JP5" gate="G$1" x="101.6" y="88.9" rot="R270"/>
+<instance part="JP6" gate="G$1" x="111.76" y="88.9" rot="R270"/>
+<instance part="JP7" gate="G$1" x="165.1" y="124.46" rot="R90"/>
+<instance part="JP8" gate="G$1" x="154.94" y="124.46" rot="R90"/>
 </instances>
 <busses>

Commit message: update layout
Parts:
- added JP10, JP11, JP12, JP9: M01SMD-6X3, SparkFun-Connectors-modified:M01SMD-6X3
Connections:
- new net GND: JP10.1, JP12.1, JP2.1, JP4.1, JP6.1, JP8.1
- new net VIN: JP1.1, JP11.1, JP3.1, JP5.1, JP7.1, JP9.1
Changed lines of the file:
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@@
 <part name="JP7" library="SparkFun-Connectors-modified" deviceset="M01" device="SMD-6X3"/>
 <part name="JP8" library="SparkFun-Connectors-modified" deviceset="M01" device="SMD-6X3"/>
+<part name="JP9" library="SparkFun-Connectors-modified" deviceset="M01" device="SMD-6X3"/>
+<part name="JP10" library="SparkFun-Connectors-modified" deviceset="M01" device="SMD-6X3"/>
+<part name="SUPPLY1" library="SparkFun-Aesthetics" deviceset="VIN" device=""/>
+<part name="GND1" library="SparkFun-Aesthetics" deviceset="GND" device=""/>
+<part name="SUPPLY2" library="SparkFun-Aesthetics" deviceset="VIN" device=""/>
+<part name="SUPPLY3" library="SparkFun-Aesthetics" deviceset="VIN" device=""/>
+<part name="SUPPLY4" library="SparkFun-Aesthetics" deviceset="VIN" device=""/>
+<part name="SUPPLY5" library="SparkFun-Aesthetics" deviceset="VIN" device=""/>
+<part name="GND2" library="SparkFun-Aesthetics" deviceset="GND" device=""/>
+<part name="GND3" library="SparkFun-Aesthetics" deviceset="GND" device=""/>
+<part name="GND4" library="SparkFun-Aesthetics" deviceset="GND" device=""/>
+<part name="GND5" library="SparkFun-Aesthetics" deviceset="GND" device=""/>
+<part name="JP11" library="SparkFun-Connectors-modified" deviceset="M01" device="SMD-6X3"/>
+<part name="JP12" library="SparkFun-Connectors-modified" deviceset="M01" device="SMD-6X3"/>
 </parts>
 <sheets>
@@
 <instance part="JP7" gate="G$1" x="165.1" y="124.46" rot="R90"/>
 <instance part="JP8" gate="G$1" x="154.94" y="124.46" rot="R90"/>
+<instance part="JP9" gate="G$1" x="71.12" y="162.56" rot="R180"/>
+<instance part="JP10" gate="G$1" x="71.12" y="152.4" rot="R180"/>
+<instance part="SUPPLY1" gate="G$1" x="58.42" y="162.56" rot="R90"/>
+<instance part="GND1" gate="1" x="55.88" y="152.4" rot="R270"/>
+<instance part="SUPPLY2" gate="G$1" x="101.6" y="134.62"/>
+<instance part="SUPPLY3" gate="G$1" x="165.1" y="134.62"/>
+<instance part="SUPPLY4" gate="G$1" x="101.6" y="78.74" rot="R180"/>
+<instance part="SUPPLY5" gate="G$1" x="165.1" y="78.74" rot="R180"/>
+<instance part="GND2" gate="1" x="111.76" y="137.16" rot="R180"/>
+<instance part="GND3" gate="1" x="154.94" y="137.16" rot="R180"/>
+<instance part="GND4" gate="1" x="111.76" y="76.2"/>
+<instance part="GND5" gate="1" x="154.94" y="76.2"/>
+<instance part="JP11" gate="G$1" x="71.12" y="172.72" rot="R180"/>
+<instance part="JP12" gate="G$1" x="71.12" y="142.24" rot="R180"/>
 </instances>
 <busses>
 </busses>
 <nets>
+<net name="VIN" class="0">
+<segment>
+<pinref part="SUPPLY1" gate="G$1" pin="VIN"/>
+<pinref part="JP9" gate="G$1" pin="1"/>
+<wire x1="58.42" y1="162.56" x2="60.96" y2="162.56" width="0.1524" layer="91"/>
+<pinref part="JP11" gate="G$1" pin="1"/>
+<wire x1="60.96" y1="162.56" x2="63.5" y2="162.56" width="0.1524" layer="91"/>
+<wire x1="63.5" y1="172.72" x2="60.96" y2="172.72" width="0.1524" layer="91"/>
+<wire x1="60.96" y1="172.72" x2="60.96" y2="162.56" width="0.1524" layer="91"/>
+<junction x="60.96" y="162.56"/>
+</segment>
+<segment>
+<pinref part="JP1" gate="G$1" pin="1"/>
+<pinref part="SUPPLY2" gate="G$1" pin="VIN"/>
+<wire x1="101.6" y1="134.62" x2="101.6" y2="132.08" width="0.1524" layer="91"/>
+</segment>
+<segment>
+<pinref part="JP7" gate="G$1" pin="1"/>
+<pinref part="SUPPLY3" gate="G$1" pin="VIN"/>
+<wire x1="165.1" y1="134.62" x2="165.1" y2="132.08" width="0.1524" layer="91"/>
+</segment>
+<segment>
+<pinref part="JP5" gate="G$1" pin="1"/>
+<pinref part="SUPPLY4" gate="G$1" pin="VIN"/>
+<wire x1="101.6" y1="78.74" x2="101.6" y2="81.28" width="0.1524" layer="91"/>
+</segment>
+<segment>
+<pinref part="JP3" gate="G$1" pin="1"/>
+<pinref part="SUPPLY5" gate="G$1" pin="VIN"/>
+<wire x1="165.1" y1="78.74" x2="165.1" y2="81.28" width="0.1524" layer="91"/>
+</segment>
+</net>
+<net name="GND" class="0">
+<segment>
+<pinref part="JP10" gate="G$1" pin="1"/>
+<pinref part="GND1" gate="1" pin="GND"/>
+<wire x1="63.5" y1="152.4" x2="60.96" y2="152.4" width="0.1524" layer="91"/>
+<pinref part="JP12" gate="G$1" pin="1"/>
+<wire x1="60.96" y1="152.4" x2="58.42" y2="152.4" width="0.1524" layer="91"/>
+<wire x1="63.5" y1="142.24" x2="60.96" y2="142.24" width="0.1524" layer="91"/>
+<wire x1="60.96" y1="142.24" x2="60.96" y2="152.4" width="0.1524" layer="91"/>
+<junction x="60.96" y="152.4"/>
+</segment>
+<segment>
+<pinref part="JP2" gate="G$1" pin="1"/>
+<pinref part="GND2" gate="1" pin="GND"/>
+<wire x1="111.76" y1="134.62" x2="111.76" y2="132.08" width="0.1524" layer="91"/>
+</segment>
+<segment>
+<pinref part="JP8" gate="G$1" pin="1"/>
+<pinref part="GND3" gate="1" pin="GND"/>
+<wire x1="154.94" y1="134.62" x2="154.94" y2="132.08" width="0.1524" layer="91"/>
+</segment>
+<segment>
+<pinref part="JP6" gate="G$1" pin="1"/>
+<pinref part="GND4" gate="1" pin="GND"/>
+<wire x1="111.76" y1="78.74" x2="111.76" y2="81.28" width="0.1524" layer="91"/>
+</segment>
+<segment>
+<pinref part="JP4" gate="G$1" pin="1"/>
+<pinref part="GND5" gate="1" pin="GND"/>
+<wire x1="154.94" y1="78.74" x2="154.94" y2="81.28" width="0.1524" layer="91"/>
+</segment>
+</net>
 </nets>
 </sheet>
