File: power.sch (EAGLE design)
At the start: 22 parts

Commit message: almost done
Parts:
- added JP13: (no value), SparkFun-Connectors:M03LONGPADS
- added JP14: M02PTH3, SparkFun-Connectors:M02PTH3
- added S2: SWITCH-MOMENTARY-2PTH-2, SparkFun-Electromechanical:SWITCH-MOMENTARY-2PTH-2
- added SAFETY: (no value), adafruit:LEDSMT1206
- added SG1: BUZZERNS, SparkFun-Electromechanical:BUZZERNS
Connections:
- new net 3.3V: JP13.1, S2.2, SAFETY.A
- new net N$3: JP14.1, SG1.1
- new net N$4: JP13.3, S2.1
- new net N$5: JP13.2, SAFETY.C
- new net N$6: JP14.2, SG1.2
Changed lines of the file:
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@@
 <setting verticaltext="up"/>
 </settings>
-<grid distance="0.1" unitdist="inch" unit="inch" style="lines" multiple="1" display="no" altdistance="0.01" altunitdist="inch" altunit="inch"/>
+<grid distance="0.1" unitdist="inch" unit="inch" style="lines" multiple="1" display="yes" altdistance="0.01" altunitdist="inch" altunit="inch"/>
 <layers>
-<layer number="1" name="Top" color="4" fill="1" visible="no" active="no"/>
-<layer number="16" name="Bottom" color="1" fill="1" visible="no" active="no"/>
-<layer number="17" name="Pads" color="2" fill="1" visible="no" active="no"/>
-<layer number="18" name="Vias" color="2" fill="1" visible="no" active="no"/>
-<layer number="19" name="Unrouted" color="6" fill="1" visible="no" active="no"/>
-<layer number="20" name="Dimension" color="15" fill="1" visible="no" active="no"/>
-<layer number="21" name="tPlace" color="7" fill="1" visible="no" active="no"/>
-<layer number="22" name="bPlace" color="7" fill="1" visible="no" active="no"/>
-<layer number="23" name="tOrigins" color="15" fill="1" visible="no" active="no"/>
-<layer number="24" name="bOrigins" color="15" fill="1" visible="no" active="no"/>
-<layer number="25" name="tNames" color="7" fill="1" visible="no" active="no"/>
-<layer number="26" name="bNames" color="7" fill="1" visible="no" active="no"/>
-<layer number="27" name="tValues" color="7" fill="1" visible="no" active="no"/>
-<layer number="28" name="bValues" color="7" fill="1" visible="no" active="no"/>
+<layer number="1" name="Top" color="4" fill="1" visible="yes" active="no"/>
+<layer number="16" name="Bottom" color="1" fill="1" visible="yes" active="no"/>
+<layer number="17" name="Pads" color="2" fill="1" visible="yes" active="no"/>
+<layer number="18" name="Vias" color="2" fill="1" visible="yes" active="no"/>
+<layer number="19" name="Unrouted" color="6" fill="1" visible="yes" active="no"/>
+<layer number="20" name="Dimension" color="15" fill="1" visible="yes" active="no"/>
+<layer number="21" name="tPlace" color="7" fill="1" visible="yes" active="no"/>
+<layer number="22" name="bPlace" color="7" fill="1" visible="yes" active="no"/>
+<layer number="23" name="tOrigins" color="15" fill="1" visible="yes" active="no"/>
+<layer number="24" name="bOrigins" color="15" fill="1" visible="yes" active="no"/>
+<layer number="25" name="tNames" color="7" fill="1" visible="yes" active="no"/>
+<layer number="26" name="bNames" color="7" fill="1" visible="yes" active="no"/>
+<layer number="27" name="tValues" color="7" fill="1" visible="yes" active="no"/>
+<layer number="28" name="bValues" color="7" fill="1" visible="yes" active="no"/>
 <layer number="29" name="tStop" color="7" fill="3" visible="no" active="no"/>
 <layer number="30" name="bStop" color="7" fill="6" visible="no" active="no"/>
@@
 <layer number="35" name="tGlue" color="7" fill="4" visible="no" active="no"/>
 <layer number="36" name="bGlue" color="7" fill="5" visible="no" active="no"/>
-<layer number="37" name="tTest" color="7" fill="1" visible="no" active="no"/>
-<layer number="38" name="bTest" color="7" fill="1" visible="no" active="no"/>
+<layer number="37" name="tTest" color="7" fill="1" visible="yes" active="no"/>
+<layer number="38" name="bTest" color="7" fill="1" visible="yes" active="no"/>
 <layer number="39" name="tKeepout" color="4" fill="11" visible="no" active="no"/>
 <layer number="40" name="bKeepout" color="1" fill="11" visible="no" active="no"/>
@@
 <layer number="44" name="Drills" color="7" fill="1" visible="no" active="no"/>
 <layer number="45" name="Holes" color="7" fill="1" visible="no" active="no"/>
-<layer number="46" name="Milling" color="3" fill="1" visible="no" active="no"/>
-<layer number="47" name="Measures" color="7" fill="1" visible="no" active="no"/>
-<layer number="48" name="Document" color="7" fill="1" visible="no" active="no"/>
-<layer number="49" name="Reference" color="7" fill="1" visible="no" active="no"/>
-<layer number="50" name="dxf" color="7" fill="1" visible="no" active="no"/>
-<layer number="51" name="tDocu" color="7" fill="1" visible="no" active="no"/>
-<layer number="52" name="bDocu" color="7" fill="1" visible="no" active="no"/>
-<layer number="53" name="tGND_GNDA" color="7" fill="9" visible="no" active="no"/>
-<layer number="54" name="bGND_GNDA" color="1" fill="9" visible="no" active="no"/>
-<layer number="56" name="wert" color="7" fill="1" visible="no" active="no"/>
-<layer number="57" name="tCAD" color="7" fill="1" visible="no" active="no"/>
+<layer number="46" name="Milling" color="3" fill="1" visible="yes" active="no"/>
+<layer number="47" name="Measures" color="7" fill="1" visible="yes" active="no"/>
+<layer number="48" name="Document" color="7" fill="1" visible="yes" active="no"/>
+<layer number="49" name="Reference" color="7" fill="1" visible="yes" active="no"/>
+<layer number="50" name="dxf" color="7" fill="1" visible="yes" active="no"/>
+<layer number="51" name="tDocu" color="7" fill="1" visible="yes" active="no"/>
+<layer number="52" name="bDocu" color="7" fill="1" visible="yes" active="no"/>
+<layer number="53" name="tGND_GNDA" color="7" fill="9" visible="yes" active="no"/>
+<layer number="54" name="bGND_GNDA" color="1" fill="9" visible="yes" active="no"/>
+<layer number="56" name="wert" color="7" fill="1" visible="yes" active="no"/>
+<layer number="57" name="tCAD" color="7" fill="1" visible="yes" active="no"/>
 <layer number="90" name="Modules" color="5" fill="1" visible="yes" active="yes"/>
 <layer number="91" name="Nets" color="2" fill="1" visible="yes" active="yes"/>
@@
 <part name="JP11" library="SparkFun-Connectors-modified" deviceset="M01" device="SMD-6X3"/>
 <part name="JP12" library="SparkFun-Connectors-modified" deviceset="M01" device="SMD-6X3"/>
+<part name="SG1" library="SparkFun-Electromechanical" deviceset="BUZZER" device="NS"/>
+<part name="SAFETY" library="adafruit" deviceset="LED" device="SMT1206"/>
+<part name="S2" library="SparkFun-Electromechanical" deviceset="SWITCH-MOMENTARY-2" device="PTH-2"/>
+<part name="JP13" library="SparkFun-Connectors" deviceset="M03" device="LONGPADS"/>
+<part name="JP14" library="SparkFun-Connectors" deviceset="M02" device="PTH3" value="M02PTH3"/>
+<part name="SUPPLY6" library="SparkFun-Aesthetics" deviceset="3.3V" device=""/>
 </parts>
 <sheets>
@@
 <instance part="JP11" gate="G$1" x="71.12" y="172.72" rot="R180"/>
 <instance part="JP12" gate="G$1" x="71.12" y="142.24" rot="R180"/>
+<instance part="SG1" gate="G$1" x="198.12" y="73.66" rot="MR0"/>
+<instance part="SAFETY" gate="G$1" x="55.88" y="60.96" rot="R90"/>
+<instance part="S2" gate="G$1" x="45.72" y="55.88"/>
+<instance part="JP13" gate="G$1" x="30.48" y="58.42" rot="MR180"/>
+<instance part="JP14" gate="G$1" x="220.98" y="63.5" rot="R180"/>
+<instance part="SUPPLY6" gate="G$1" x="48.26" y="68.58"/>
 </instances>
 <busses>
@@
 </segment>
 </net>
+<net name="3.3V" class="0">
+<segment>
+<pinref part="SAFETY" gate="G$1" pin="A"/>
+<pinref part="SUPPLY6" gate="G$1" pin="3.3V"/>
+<wire x1="48.26" y1="60.96" x2="48.26" y2="63.5" width="0.1524" layer="91"/>
+<wire x1="48.26" y1="63.5" x2="48.26" y2="68.58" width="0.1524" layer="91"/>
+<wire x1="48.26" y1="60.96" x2="53.34" y2="60.96" width="0.1524" layer="91"/>
+<junction x="48.26" y="60.96"/>
+<pinref part="JP13" gate="G$1" pin="1"/>
+<wire x1="38.1" y1="60.96" x2="48.26" y2="60.96" width="0.1524" layer="91"/>
+<pinref part="S2" gate="G$1" pin="2"/>
+<wire x1="50.8" y1="55.88" x2="66.04" y2="55.88" width="0.1524" layer="91"/>
+<wire x1="66.04" y1="55.88" x2="66.04" y2="63.5" width="0.1524" layer="91"/>
+<wire x1="66.04" y1="63.5" x2="48.26" y2="63.5" width="0.1524" layer="91"/>
+<junction x="48.26" y="63.5"/>
+</segment>
+</net>
+<net name="N$5" class="0">
+<segment>
+<pinref part="SAFETY" gate="G$1" pin="C"/>
+<wire x1="60.96" y1="60.96" x2="63.5" y2="60.96" width="0.1524" layer="91"/>
+<wire x1="63.5" y1="60.96" x2="63.5" y2="58.42" width="0.1524" layer="91"/>
+<pinref part="JP13" gate="G$1" pin="2"/>
+<wire x1="63.5" y1="58.42" x2="38.1" y2="58.42" width="0.1524" layer="91"/>
+</segment>
+</net>
+<net name="N$6" class="0">
+<segment>
+<pinref part="SG1" gate="G$1" pin="2"/>
+<wire x1="195.58" y1="60.96" x2="195.58" y2="71.12" width="0.1524" layer="91"/>
+<pinref part="JP14" gate="G$1" pin="2"/>
+<wire x1="195.58" y1="60.96" x2="213.36" y2="60.96" width="0.1524" layer="91"/>
+</segment>
+</net>
+<net name="N$3" class="0">
+<segment>
+<pinref part="JP14" gate="G$1" pin="1"/>
+<pinref part="SG1" gate="G$1" pin="1"/>
+<wire x1="213.36" y1="63.5" x2="198.12" y2="63.5" width="0.1524" layer="91"/>
+<wire x1="198.12" y1="63.5" x2="198.12" y2="71.12" width="0.1524" layer="91"/>
+</segment>
+</net>
+<net name="N$4" class="0">
+<segment>
+<pinref part="JP13" gate="G$1" pin="3"/>
+<pinref part="S2" gate="G$1" pin="1"/>
+<wire x1="38.1" y1="55.88" x2="40.64" y2="55.88" width="0.1524" layer="91"/>
+</segment>
+</net>

Commit message: basically done
Parts:
- added JP15, JP16: M01SMD, SparkFun-Connectors-modified:M01SMD
- SAFETY: device adafruit:LEDSMT1206 -> adafruit:LED5MM
Connections:
- net N$3: now also JP16.1
- net N$6: now also JP15.1
Other:
- moved on the sheet: SG1
Changed lines of the file:
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@@
 <part name="JP12" library="SparkFun-Connectors-modified" deviceset="M01" device="SMD-6X3"/>
 <part name="SG1" library="SparkFun-Electromechanical" deviceset="BUZZER" device="NS"/>
-<part name="SAFETY" library="adafruit" deviceset="LED" device="SMT1206"/>
+<part name="SAFETY" library="adafruit" deviceset="LED" device="5MM"/>
 <part name="S2" library="SparkFun-Electromechanical" deviceset="SWITCH-MOMENTARY-2" device="PTH-2"/>
 <part name="JP13" library="SparkFun-Connectors" deviceset="M03" device="LONGPADS"/>
 <part name="JP14" library="SparkFun-Connectors" deviceset="M02" device="PTH3" value="M02PTH3"/>
 <part name="SUPPLY6" library="SparkFun-Aesthetics" deviceset="3.3V" device=""/>
+<part name="JP15" library="SparkFun-Connectors-modified" deviceset="M01" device="SMD" value="M01SMD"/>
+<part name="JP16" library="SparkFun-Connectors-modified" deviceset="M01" device="SMD" value="M01SMD"/>
 </parts>
 <sheets>
@@
 <instance part="JP11" gate="G$1" x="71.12" y="172.72" rot="R180"/>
 <instance part="JP12" gate="G$1" x="71.12" y="142.24" rot="R180"/>
-<instance part="SG1" gate="G$1" x="198.12" y="73.66" rot="MR0"/>
+<instance part="SG1" gate="G$1" x="198.12" y="96.52" rot="MR0"/>
 <instance part="SAFETY" gate="G$1" x="55.88" y="60.96" rot="R90"/>
 <instance part="S2" gate="G$1" x="45.72" y="55.88"/>
@@
 <instance part="JP14" gate="G$1" x="220.98" y="63.5" rot="R180"/>
 <instance part="SUPPLY6" gate="G$1" x="48.26" y="68.58"/>
+<instance part="JP15" gate="G$1" x="220.98" y="76.2" rot="R180"/>
+<instance part="JP16" gate="G$1" x="220.98" y="86.36" rot="R180"/>
 </instances>
 <busses>
@@
 <segment>
 <pinref part="SG1" gate="G$1" pin="2"/>
-<wire x1="195.58" y1="60.96" x2="195.58" y2="71.12" width="0.1524" layer="91"/>
+<wire x1="195.58" y1="60.96" x2="195.58" y2="76.2" width="0.1524" layer="91"/>
 <pinref part="JP14" gate="G$1" pin="2"/>
+<wire x1="195.58" y1="76.2" x2="195.58" y2="93.98" width="0.1524" layer="91"/>
 <wire x1="195.58" y1="60.96" x2="213.36" y2="60.96" width="0.1524" layer="91"/>
+<pinref part="JP15" gate="G$1" pin="1"/>
+<wire x1="213.36" y1="76.2" x2="195.58" y2="76.2" width="0.1524" layer="91"/>
+<junction x="195.58" y="76.2"/>
 </segment>
 </net>
@@
 <pinref part="SG1" gate="G$1" pin="1"/>
 <wire x1="213.36" y1="63.5" x2="198.12" y2="63.5" width="0.1524" layer="91"/>
-<wire x1="198.12" y1="63.5" x2="198.12" y2="71.12" width="0.1524" layer="91"/>
+<wire x1="198.12" y1="63.5" x2="198.12" y2="86.36" width="0.1524" layer="91"/>
+<pinref part="JP16" gate="G$1" pin="1"/>
+<wire x1="198.12" y1="86.36" x2="198.12" y2="93.98" width="0.1524" layer="91"/>
+<wire x1="213.36" y1="86.36" x2="198.12" y2="86.36" width="0.1524" layer="91"/>
+<junction x="198.12" y="86.36"/>
+<wire x1="213.36" y1="86.36" x2="198.12" y2="86.36" width="0.1524" layer="91"/>
+<wire x1="213.36" y1="86.36" x2="198.12" y2="86.36" width="0.1524" layer="91"/>
 </segment>
 </net>
